File: stm32_encoderXY_imu.brd (EAGLE design)
At the start: 100.3 x 86 mm, 16 parts

Commit message: init
Parts:
- moved SER3 5.62 mm to (31.1, 75.9)
- moved ENC2 2.54 mm to (88.9, 48.8)
- moved VIN 2.54 mm to (88.9, 34.6), flipped to the top
- moved SER1 1.94 mm to (12.2, 76.1)
- moved ENC1 1.27 mm to (60.5, 76.2)
Connections:
- net PA_2: no longer ENC1.4
- net PA_3: no longer ENC1.3
- net PA_6: now also ENC1.4
- net PA_7: now also ENC1.3
Routing:
- net GND: track 284.3 -> 399.2 mm
- net PA_6: track 13.2 -> 49.2 mm
- net PA_7: track 13.2 -> 49.2 mm
- net PA_2: track 39.2 -> 13.3 mm
- net PA_3: track 37.8 -> 13.2 mm
- net 5V: track 207.9 -> 199.1 mm, vias 5 -> 1
- net PB_11: track 36.0 -> 28.4 mm
- net PB_10: track 35.3 -> 28.4 mm
- net PA_10: track 64.6 -> 70.4 mm
- net PA_9: track 65.2 -> 70.7 mm
- net PB_7: track 98.8 -> 96.0 mm
- net PA_1: track 61.5 -> 59.0 mm
- net PA_0: track 57.2 -> 54.7 mm
- net PB_6: track 94.1 -> 96.6 mm
- net PB_12: track 12.2 -> 11.6 mm
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Other:
- board text added: "IMU"
