File: stm32_encoderXY_imu.sch (EAGLE design)
At the start: 16 parts

Commit message: init
Connections:
- net PA_2: no longer ENC1.SIG2
- net PA_3: no longer ENC1.SIG1
- net PA_6: now also ENC1.SIG2
- net PA_7: now also ENC1.SIG1
Other:
- moved on the sheet: JP1, JP2
